File: ble-audio-adapter.sch (KiCad schematic (older format))
At the start: 24 parts, among them P1 AUDIO_JACK_CONN, P2 PWR_SW_CONN, P3 PAIR_BTN_CONN, P4 PLAY/PAUSE_BTN, P5 VOL_UP_BTN, P6 VOL_DOWN_BTN

Commit message: Updated reference positioning
Parts:
- BT1: value Battery -> 9V; footprint (none) -> component_footprints:Battery_Connector
Changed lines of the file:
@@
 LIBS:ble_uart_friend
 LIBS:KL05
-LIBS:ble-audio-adapter-cache
+LIBS:74xgxx
+LIBS:ac-dc
+LIBS:actel
+LIBS:Altera
+LIBS:analog_devices
+LIBS:brooktre
+LIBS:cmos_ieee
+LIBS:dc-dc
+LIBS:diode
+LIBS:elec-unifil
+LIBS:ESD_Protection
+LIBS:ftdi
+LIBS:gennum
+LIBS:graphic
+LIBS:hc11
+LIBS:ir
+LIBS:Lattice
+LIBS:logo
+LIBS:maxim
+LIBS:microchip_dspic33dsc
+LIBS:microchip_pic10mcu
+LIBS:microchip_pic12mcu
+LIBS:microchip_pic16mcu
+LIBS:microchip_pic18mcu
+LIBS:microchip_pic32mcu
+LIBS:motor_drivers
+LIBS:msp430
+LIBS:nordicsemi
+LIBS:nxp_armmcu
+LIBS:onsemi
+LIBS:Oscillators
+LIBS:powerint
+LIBS:Power_Management
+LIBS:pspice
+LIBS:references
+LIBS:relays
+LIBS:rfcom
+LIBS:sensors
+LIBS:silabs
+LIBS:stm8
+LIBS:stm32
+LIBS:supertex
+LIBS:switches
+LIBS:transf
+LIBS:ttl_ieee
+LIBS:video
+LIBS:Xicor
+LIBS:Zilog
 EELAYER 25 0
 EELAYER END
@@
 P 5500 1600
 F 0 "BT1" H 5600 1650 50  0000 L CNN
-F 1 "Battery" H 5550 1500 50  0000 L CNN
-F 2 "" V 5500 1640 50  0001 C CNN
+F 1 "9V" H 5300 1600 50  0000 L CNN
+F 2 "component_footprints:Battery_Connector" V 5500 1640 50  0001 C CNN
 F 3 "" V 5500 1640 50  0000 C CNN
 	1    5500 1600
